Commit message: update robot description for my-bot pkg

File: description/robot_core.xacro (robot description, xacro)
@@ -23,23 +23,23 @@
         <parent link="base_link" />
         <child link="chassis" />
-        <origin xyz="-0.1 0 0" />
+        <origin xyz="-0.25 0 -0.0175" />
     </joint>
     <!-- CHASSIS LINK -->
     <link name="chassis">
         <visual>
-            <origin xyz="0.15 0 0.075" />
+            <origin xyz="0.25 0 0.075" />
             <geometry>
-                <box size="0.3 0.3 0.15" />
+                <box size="0.5 0.4 0.15" />
             </geometry>
             <material name="white" />
         </visual>
         <collision>
-            <origin xyz="0.15 0 0.075" />
+            <origin xyz="0.25 0 0.075" />
             <geometry>
-                <box size="0.3 0.3 0.15" />
+                <box size="0.5 0.4 0.15" />
             </geometry>
         </collision>
-        <xacro:inertial_box mass="0.5" x="0.3" y="0.3" z="0.15">
-            <origin xyz="0.15 0.15 0.075" rpy="0 0 0" />
+        <xacro:inertial_box mass="0.5" x="0.5" y="0.4" z="0.15">
+            <origin xyz="0.25 0.2 0.075" rpy="0 0 0" />
         </xacro:inertial_box>
     </link>
@@ -53,5 +53,5 @@
         <parent link="base_link" />
         <child link="left_wheel" />
-        <origin xyz="0 0.175 0" rpy="-${pi/2} 0 0" />
+        <origin xyz="0 0.22 0" rpy="-${pi/2} 0 0" />
         <axis xyz="0 0 1" />
     </joint>
@@ -59,5 +59,5 @@
         <visual>
             <geometry>
-                <cylinder radius="0.05" length="0.04" />
+                <cylinder radius="0.045" length="0.015" />
             </geometry>
             <material name="blue" />
@@ -65,8 +65,8 @@
         <collision>
             <geometry>
-                <cylinder radius="0.05" length="0.04" />
+                <cylinder radius="0.045" length="0.015" />
             </geometry>
         </collision>
-        <xacro:inertial_cylinder mass="0.1" length="0.04" radius="0.05">
+        <xacro:inertial_cylinder mass="0.1" length="0.015" radius="0.045">
             <origin xyz="0 0 0" rpy="0 0 0" />
         </xacro:inertial_cylinder>
@@ -81,5 +81,5 @@
         <parent link="base_link" />
         <child link="right_wheel" />
-        <origin xyz="0 -0.175 0" rpy="${pi/2} 0 0" />
+        <origin xyz="0 -0.22 0" rpy="${pi/2} 0 0" />
         <axis xyz="0 0 -1" />
     </joint>
@@ -87,5 +87,5 @@
         <visual>
             <geometry>
-                <cylinder radius="0.05" length="0.04" />
+                <cylinder radius="0.045" length="0.015" />
             </geometry>
             <material name="blue" />
@@ -93,8 +93,8 @@
         <collision>
             <geometry>
-                <cylinder radius="0.05" length="0.04" />
+                <cylinder radius="0.045" length="0.015" />
             </geometry>
         </collision>
-        <xacro:inertial_cylinder mass="0.1" length="0.04" radius="0.05">
+        <xacro:inertial_cylinder mass="0.1" length="0.015" radius="0.045">
             <origin xyz="0 0 0" rpy="0 0 0" />
         </xacro:inertial_cylinder>
@@ -106,13 +106,13 @@
     </gazebo>
     <!-- CASTER WHEEL -->
-    <joint name="caster_wheel_joint" type="fixed">
+    <joint name="caster_wheel_fontleft_joint" type="fixed">
         <parent link="chassis" />
-        <child link="caster_wheel" />
-        <origin xyz="0.24 0 0" />
+        <child link="caster_wheel_fontleft" />
+        <origin xyz="0.4 0.15 0" />
     </joint>
-    <link name="caster_wheel">
+    <link name="caster_wheel_fontleft">
         <visual>
             <geometry>
-                <sphere radius="0.05" />
+                <sphere radius="0.03" />
             </geometry>
             <material name="black" />
@@ -120,12 +120,12 @@
         <collision>
             <geometry>
-                <sphere radius="0.05" />
+                <sphere radius="0.03" />
             </geometry>
         </collision>
-        <xacro:inertial_sphere mass="0.1" radius="0.05">
+        <xacro:inertial_sphere mass="0.03" radius="0.03">
             <origin xyz="0 0 0" rpy="0 0 0" />
         </xacro:inertial_sphere>
     </link>
-    <gazebo reference="caster_wheel">
+    <gazebo reference="caster_wheel_fontleft">
         <material>
             Gazebo/Black
